File: PoE_supply.kicad_sch (KiCad schematic)
At the start: 23 parts, among them J1 Bus_RJ45_5-2337992-8, Q1 PJE138K, U1 TPS2372-3RGWR, U4 IEA48003A280V-001-R

Commit message: [#62835] Change dcdc placement, change IC's placement
Connections:
- net P1 renamed MDI0_P
- net P10 renamed MDI3_N
- net P2 renamed MDI0_N
- net P3 renamed MDI1_P
- net P6 renamed MDI1_N
- net P7 renamed MDI2_P
- net P8 renamed MDI2_N
- net P9 renamed MDI3_P
Changed lines of the file:
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@@
 (kicad_sch (version 20230121) (generator eeschema)
   (paper "A3")
+  (bus_alias "ETH" (members "MDI0_P" "MDI0_N" "MDI1_P" "MDI1_N" "MDI2_P" "MDI2_N" "MDI3_N" "MDI3_P"))
   (junction (at 210.185 134.62) (diameter 0) (color 0 0 0 0)
   )
@@
     (stroke (width 0) (type default))
   )
-  (wire (pts (xy 107.95 106.68) (xy 114.3 106.68))
-    (stroke (width 0) (type default))
-  )
-  (wire (pts (xy 39.37 31.75) (xy 43.18 31.75))
-    (stroke (width 0) (type default))
-  )
-  (wire (pts (xy 39.37 26.67) (xy 43.18 26.67))
+  (wire (pts (xy 107.95 106.68) (xy 117.475 106.68))
+    (stroke (width 0) (type default))
+  )
+  (wire (pts (xy 39.37 31.75) (xy 48.26 31.75))
+    (stroke (width 0) (type default))
+  )
+  (wire (pts (xy 39.37 26.67) (xy 48.26 26.67))
     (stroke (width 0) (type default))
   )
@@
     (stroke (width 0) (type default))
   )
-  (wire (pts (xy 107.95 114.3) (xy 114.3 114.3))
+  (wire (pts (xy 107.95 114.3) (xy 117.475 114.3))
     (stroke (width 0) (type default))
   )
@@
     (stroke (width 0) (type default))
   )
-  (wire (pts (xy 107.95 109.22) (xy 114.3 109.22))
+  (wire (pts (xy 107.95 109.22) (xy 117.475 109.22))
     (stroke (width 0) (type default))
   )
@@
     (stroke (width 0) (type default))
   )
-  (wire (pts (xy 39.37 44.45) (xy 43.18 44.45))
+  (wire (pts (xy 39.37 44.45) (xy 48.26 44.45))
     (stroke (width 0) (type default))
   )
@@
     (stroke (width 0) (type default))
   )
-  (wire (pts (xy 107.95 119.38) (xy 114.3 119.38))
+  (wire (pts (xy 107.95 119.38) (xy 117.475 119.38))
     (stroke (width 0) (type default))
   )
@@
     (stroke (width 0) (type default))
   )
-  (wire (pts (xy 107.95 111.76) (xy 114.3 111.76))
+  (wire (pts (xy 107.95 111.76) (xy 117.475 111.76))
     (stroke (width 0) (type default))
   )
@@
     (stroke (width 0) (type default))
   )
-  (wire (pts (xy 39.37 39.37) (xy 43.18 39.37))
+  (wire (pts (xy 39.37 39.37) (xy 48.26 39.37))
     (stroke (width 0) (type default))
   )
@@
     (stroke (width 0) (type default))
   )
-  (wire (pts (xy 39.37 36.83) (xy 43.18 36.83))
+  (wire (pts (xy 39.37 36.83) (xy 48.26 36.83))
     (stroke (width 0) (type default))
   )
@@
     (stroke (width 0) (type default))
   )
-  (wire (pts (xy 39.37 29.21) (xy 43.18 29.21))
+  (wire (pts (xy 39.37 29.21) (xy 48.26 29.21))
     (stroke (width 0) (type default))
   )
@@
     (stroke (width 0) (type default))
   )
-  (wire (pts (xy 39.37 34.29) (xy 43.18 34.29))
+  (wire (pts (xy 39.37 34.29) (xy 48.26 34.29))
     (stroke (width 0) (type default))
   )
@@
     (stroke (width 0) (type default))
   )
-  (wire (pts (xy 39.37 41.91) (xy 43.18 41.91))
+  (wire (pts (xy 39.37 41.91) (xy 48.26 41.91))
     (stroke (width 0) (type default))
   )
@@
     (stroke (width 0) (type default))
   )
-  (wire (pts (xy 107.95 121.92) (xy 114.3 121.92))
-    (stroke (width 0) (type default))
-  )
-  (wire (pts (xy 107.95 104.14) (xy 114.3 104.14))
+  (wire (pts (xy 107.95 121.92) (xy 117.475 121.92))
+    (stroke (width 0) (type default))
+  )
+  (wire (pts (xy 107.95 104.14) (xy 117.475 104.14))
     (stroke (width 0) (type default))
   )
@@
     (stroke (width 0) (type default))
   )
-  (wire (pts (xy 107.95 116.84) (xy 114.3 116.84))
+  (wire (pts (xy 107.95 116.84) (xy 117.475 116.84))
     (stroke (width 0) (type default))
   )
@@
     (effects (font (size 1.27 1.27)) (justify left bottom))
   )
-  (label "P7" (at 43.18 36.83 180) (fields_autoplaced)
-    (effects (font (size 1.27 1.27)) (justify right bottom))
-  )
   (label "VC1" (at 114.3 132.08 180) (fields_autoplaced)
     (effects (font (size 1.27 1.27)) (justify right bottom))
   )
+  (label "MDI2_N" (at 117.475 116.84 180) (fields_autoplaced)
+    (effects (font (size 1.27 1.27)) (justify right bottom))
+  )
+  (label "MDI1_N" (at 48.26 34.29 180) (fields_autoplaced)
+    (effects (font (size 1.27 1.27)) (justify right bottom))
+  )
   (label "VC3" (at 114.3 137.16 180) (fields_autoplaced)
     (effects (font (size 1.27 1.27)) (justify right bottom))
@@
     (effects (font (size 1.27 1.27)) (justify left bottom))
   )
+  (label "MDI3_P" (at 117.475 119.38 180) (fields_autoplaced)
+    (effects (font (size 1.27 1.27)) (justify right bottom))
+  )
+  (label "MDI0_N" (at 117.475 106.68 180) (fields_autoplaced)
+    (effects (font (size 1.27 1.27)) (justify right bottom))
+  )
   (label "VC1" (at 139.065 102.87 0) (fields_autoplaced)
     (effects (font (size 1.27 1.27)) (justify left bottom))
   )
-  (label "P10" (at 43.18 44.45 180) (fields_autoplaced)
-    (effects (font (size 1.27 1.27)) (justify right bottom))
-  )
-  (label "P2" (at 43.18 29.21 180) (fields_autoplaced)
-    (effects (font (size 1.27 1.27)) (justify right bottom))
-  )
-  (label "P7" (at 114.3 114.3 180) (fields_autoplaced)
+  (label "MDI3_P" (at 48.26 41.91 180) (fields_autoplaced)
+    (effects (font (size 1.27 1.27)) (justify right bottom))
+  )
+  (label "MDI1_P" (at 117.475 109.22 180) (fields_autoplaced)
     (effects (font (size 1.27 1.27)) (justify right bottom))
   )
@@
     (effects (font (size 1.27 1.27)) (justify left bottom))
   )
-  (label "P3" (at 43.18 31.75 180) (fields_autoplaced)
-    (effects (font (size 1.27 1.27)) (justify right bottom))
-  )
-  (label "P6" (at 43.18 34.29 180) (fields_autoplaced)
-    (effects (font (size 1.27 1.27)) (justify right bottom))
-  )
   (label "VC2" (at 114.3 134.62 180) (fields_autoplaced)
     (effects (font (size 1.27 1.27)) (justify right bottom))
@@
     (effects (font (size 1.27 1.27)) (justify left bottom))
   )
-  (label "P10" (at 114.3 121.92 180) (fields_autoplaced)
-    (effects (font (size 1.27 1.27)) (justify right bottom))
-  )
-  (label "P1" (at 114.3 104.14 180) (fields_autoplaced)
-    (effects (font (size 1.27 1.27)) (justify right bottom))
-  )
-  (label "P1" (at 43.18 26.67 180) (fields_autoplaced)
+  (label "MDI2_P" (at 117.475 114.3 180) (fields_autoplaced)
+    (effects (font (size 1.27 1.27)) (justify right bottom))
+  )
+  (label "MDI0_P" (at 117.475 104.14 180) (fields_autoplaced)
     (effects (font (size 1.27 1.27)) (justify right bottom))
   )
@@
     (effects (font (size 1.27 1.27)) (justify left bottom))
   )
-  (label "P9" (at 114.3 119.38 180) (fields_autoplaced)
+  (label "MDI3_N" (at 117.475 121.92 180) (fields_autoplaced)
     (effects (font (size 1.27 1.27)) (justify right bottom))
   )
@@
     (effects (font (size 1.27 1.27)) (justify right bottom))
   )
+  (label "MDI2_N" (at 48.26 39.37 180) (fields_autoplaced)
+    (effects (font (size 1.27 1.27)) (justify right bottom))
+  )
+  (label "MDI1_N" (at 117.475 111.76 180) (fields_autoplaced)
+    (effects (font (size 1.27 1.27)) (justify right bottom))
+  )
   (label "VC4" (at 114.3 139.7 180) (fields_autoplaced)
     (effects (font (size 1.27 1.27)) (justify right bottom))
   )
-  (label "P9" (at 43.18 41.91 180) (fields_autoplaced)
-    (effects (font (size 1.27 1.27)) (justify right bottom))
-  )
   (label "CLSB" (at 216.535 127 0) (fields_autoplaced)
     (effects (font (size 1.27 1.27)) (justify left bottom))
   )
-  (label "P8" (at 43.18 39.37 180) (fields_autoplaced)
-    (effects (font (size 1.27 1.27)) (justify right bottom))
-  )
-  (label "P6" (at 114.3 111.76 180) (fields_autoplaced)
-    (effects (font (size 1.27 1.27)) (justify right bottom))
-  )
-  (label "P8" (at 114.3 116.84 180) (fields_autoplaced)
-    (effects (font (size 1.27 1.27)) (justify right bottom))
-  )
-  (label "P3" (at 114.3 109.22 180) (fields_autoplaced)
+  (label "MDI0_N" (at 48.26 29.21 180) (fields_autoplaced)
+    (effects (font (size 1.27 1.27)) (justify right bottom))
+  )
+  (label "MDI3_N" (at 48.26 44.45 180) (fields_autoplaced)
+    (effects (font (size 1.27 1.27)) (justify right bottom))
+  )
+  (label "MDI1_P" (at 48.26 31.75 180) (fields_autoplaced)
+    (effects (font (size 1.27 1.27)) (justify right bottom))
+  )
+  (label "MDI0_P" (at 48.26 26.67 180) (fields_autoplaced)
+    (effects (font (size 1.27 1.27)) (justify right bottom))
+  )
+  (label "MDI2_P" (at 48.26 36.83 180) (fields_autoplaced)
     (effects (font (size 1.27 1.27)) (justify right bottom))
   )
@@
     (effects (font (size 1.27 1.27)) (justify left bottom))
   )
-  (label "P2" (at 114.3 106.68 180) (fields_autoplaced)
-    (effects (font (size 1.27 1.27)) (justify right bottom))
-  )
   (hierarchical_label "{ETH}" (shape output) (at 26.67 22.86 180) (fields_autoplaced)
