File: USBPD_output.kicad_sch (KiCad schematic)
At the start: 26 parts, among them J2 Bus_RJ45_7499111121A, J3 USB-C_GCT_USB4105-GF-A, U3 INA230AIRGTR, U6 TPS65987DDHRSHR

Commit message: [#62835] Change dcdc placement, change IC's placement
Connections:
- net P1 renamed MDI0_P
- net P10 renamed MDI3_N
- net P2 renamed MDI0_N
- net P3 renamed MDI1_P
- net P6 renamed MDI1_N
- net P7 renamed MDI2_P
- net P8 renamed MDI2_N
- net P9 renamed MDI3_P
Changed lines of the file:
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@@
     (stroke (width 0) (type default))
   )
-  (wire (pts (xy 261.62 81.28) (xy 256.54 81.28))
-    (stroke (width 0) (type default))
-  )
-  (wire (pts (xy 312.42 63.5) (xy 307.34 63.5))
+  (wire (pts (xy 316.23 63.5) (xy 307.34 63.5))
     (stroke (width 0) (type default))
   )
@@
     (stroke (width 0) (type default))
   )
-  (wire (pts (xy 312.42 73.66) (xy 307.34 73.66))
+  (wire (pts (xy 316.23 73.66) (xy 307.34 73.66))
     (stroke (width 0) (type default))
   )
@@
     (stroke (width 0) (type default))
   )
-  (wire (pts (xy 261.62 86.36) (xy 256.54 86.36))
+  (wire (pts (xy 261.62 86.36) (xy 253.365 86.36))
     (stroke (width 0) (type default))
   )
@@
     (stroke (width 0) (type default))
   )
-  (wire (pts (xy 312.42 60.96) (xy 307.34 60.96))
+  (wire (pts (xy 316.23 60.96) (xy 307.34 60.96))
     (stroke (width 0) (type default))
   )
@@
     (stroke (width 0) (type default))
   )
-  (wire (pts (xy 312.42 66.04) (xy 307.34 66.04))
+  (wire (pts (xy 316.23 66.04) (xy 307.34 66.04))
     (stroke (width 0) (type default))
   )
@@
     (stroke (width 0) (type default))
   )
-  (wire (pts (xy 261.62 96.52) (xy 256.54 96.52))
+  (wire (pts (xy 261.62 96.52) (xy 253.365 96.52))
     (stroke (width 0) (type default))
   )
@@
     (stroke (width 0) (type default))
   )
-  (wire (pts (xy 261.62 91.44) (xy 256.54 91.44))
+  (wire (pts (xy 261.62 91.44) (xy 253.365 91.44))
     (stroke (width 0) (type default))
   )
@@
     (stroke (width 0) (type default))
   )
-  (wire (pts (xy 261.62 83.82) (xy 256.54 83.82))
-    (stroke (width 0) (type default))
-  )
-  (wire (pts (xy 261.62 93.98) (xy 256.54 93.98))
+  (wire (pts (xy 261.62 83.82) (xy 253.365 83.82))
+    (stroke (width 0) (type default))
+  )
+  (wire (pts (xy 261.62 93.98) (xy 253.365 93.98))
     (stroke (width 0) (type default))
   )
@@
     (stroke (width 0) (type default))
   )
-  (wire (pts (xy 312.42 58.42) (xy 307.34 58.42))
-    (stroke (width 0) (type default))
-  )
-  (wire (pts (xy 261.62 88.9) (xy 256.54 88.9))
+  (wire (pts (xy 316.23 58.42) (xy 307.34 58.42))
+    (stroke (width 0) (type default))
+  )
+  (wire (pts (xy 261.62 88.9) (xy 253.365 88.9))
     (stroke (width 0) (type default))
   )
@@
     (stroke (width 0) (type default))
   )
-  (wire (pts (xy 261.62 99.06) (xy 256.54 99.06))
+  (wire (pts (xy 261.62 99.06) (xy 253.365 99.06))
     (stroke (width 0) (type default))
   )
@@
     (stroke (width 0) (type default))
   )
-  (wire (pts (xy 312.42 71.12) (xy 307.34 71.12))
+  (wire (pts (xy 316.23 71.12) (xy 307.34 71.12))
     (stroke (width 0) (type default))
   )
@@
     (stroke (width 0) (type default))
   )
-  (wire (pts (xy 312.42 68.58) (xy 307.34 68.58))
+  (wire (pts (xy 316.23 68.58) (xy 307.34 68.58))
     (stroke (width 0) (type default))
   )
@@
     (stroke (width 0) (type default))
   )
-  (wire (pts (xy 312.42 55.88) (xy 307.34 55.88))
+  (wire (pts (xy 316.23 55.88) (xy 307.34 55.88))
     (stroke (width 0) (type default))
   )
@@
   )
   (wire (pts (xy 93.345 210.82) (xy 93.345 220.345))
+    (stroke (width 0) (type default))
+  )
+  (wire (pts (xy 253.365 81.28) (xy 261.62 81.28))
     (stroke (width 0) (type default))
   )
@@
     (effects (font (size 1.27 1.27)) (justify right bottom))
   )
+  (label "MDI2_P" (at 316.23 66.04 180) (fields_autoplaced)
+    (effects (font (size 1.27 1.27)) (justify right bottom))
+  )
   (label "D-" (at 294.64 203.2 0) (fields_autoplaced)
     (effects (font (size 1.27 1.27)) (justify left bottom))
   )
-  (label "P10" (at 256.54 99.06 0) (fields_autoplaced)
-    (effects (font (size 1.27 1.27)) (justify left bottom))
-  )
-  (label "P9" (at 256.54 96.52 0) (fields_autoplaced)
-    (effects (font (size 1.27 1.27)) (justify left bottom))
-  )
-  (label "P3" (at 312.42 60.96 180) (fields_autoplaced)
-    (effects (font (size 1.27 1.27)) (justify right bottom))
-  )
-  (label "P1" (at 312.42 55.88 180) (fields_autoplaced)
+  (label "MDI1_P" (at 253.365 86.36 0) (fields_autoplaced)
+    (effects (font (size 1.27 1.27)) (justify left bottom))
+  )
+  (label "MDI0_P" (at 316.23 55.88 180) (fields_autoplaced)
     (effects (font (size 1.27 1.27)) (justify right bottom))
   )
@@
     (effects (font (size 1.27 1.27)) (justify right bottom))
   )
-  (label "P3" (at 256.54 86.36 0) (fields_autoplaced)
-    (effects (font (size 1.27 1.27)) (justify left bottom))
-  )
-  (label "P8" (at 256.54 93.98 0) (fields_autoplaced)
-    (effects (font (size 1.27 1.27)) (justify left bottom))
+  (label "MDI1_N" (at 316.23 63.5 180) (fields_autoplaced)
+    (effects (font (size 1.27 1.27)) (justify right bottom))
   )
   (label "SDA" (at 132.08 222.25 0) (fields_autoplaced)
@@
     (effects (font (size 1.27 1.27)) (justify left bottom))
   )
-  (label "P7" (at 312.42 66.04 180) (fields_autoplaced)
-    (effects (font (size 1.27 1.27)) (justify right bottom))
-  )
-  (label "P1" (at 256.54 81.28 0) (fields_autoplaced)
-    (effects (font (size 1.27 1.27)) (justify left bottom))
-  )
-  (label "P6" (at 256.54 88.9 0) (fields_autoplaced)
-    (effects (font (size 1.27 1.27)) (justify left bottom))
-  )
-  (label "P8" (at 312.42 68.58 180) (fields_autoplaced)
-    (effects (font (size 1.27 1.27)) (justify right bottom))
+  (label "MDI1_P" (at 316.23 60.96 180) (fields_autoplaced)
+    (effects (font (size 1.27 1.27)) (justify right bottom))
+  )
+  (label "MDI3_P" (at 253.365 96.52 0) (fields_autoplaced)
+    (effects (font (size 1.27 1.27)) (justify left bottom))
+  )
+  (label "MDI0_N" (at 253.365 83.82 0) (fields_autoplaced)
+    (effects (font (size 1.27 1.27)) (justify left bottom))
   )
   (label "D+" (at 326.39 147.32 180) (fields_autoplaced)
@@
     (effects (font (size 1.27 1.27)) (justify right bottom))
   )
+  (label "MDI2_P" (at 253.365 91.44 0) (fields_autoplaced)
+    (effects (font (size 1.27 1.27)) (justify left bottom))
+  )
+  (label "MDI3_P" (at 316.23 71.12 180) (fields_autoplaced)
+    (effects (font (size 1.27 1.27)) (justify right bottom))
+  )
   (label "SCL" (at 101.6 210.82 270) (fields_autoplaced)
     (effects (font (size 1.27 1.27)) (justify right bottom))
   )
+  (label "MDI0_P" (at 253.365 81.28 0) (fields_autoplaced)
+    (effects (font (size 1.27 1.27)) (justify left bottom))
+  )
   (label "SDA" (at 118.11 210.185 270) (fields_autoplaced)
     (effects (font (size 1.27 1.27)) (justify right bottom))
@@
     (effects (font (size 1.27 1.27)) (justify right bottom))
   )
+  (label "MDI0_N" (at 316.23 58.42 180) (fields_autoplaced)
+    (effects (font (size 1.27 1.27)) (justify right bottom))
+  )
+  (label "MDI1_N" (at 253.365 88.9 0) (fields_autoplaced)
+    (effects (font (size 1.27 1.27)) (justify left bottom))
+  )
   (label "SDA" (at 97.155 210.82 270) (fields_autoplaced)
     (effects (font (size 1.27 1.27)) (justify right bottom))
@@
     (effects (font (size 1.27 1.27)) (justify right bottom))
   )
-  (label "P6" (at 312.42 63.5 180) (fields_autoplaced)
+  (label "MDI2_N" (at 316.23 68.58 180) (fields_autoplaced)
     (effects (font (size 1.27 1.27)) (justify right bottom))
   )
@@
     (effects (font (size 1.27 1.27)) (justify left bottom))
   )
-  (label "P9" (at 312.42 71.12 180) (fields_autoplaced)
-    (effects (font (size 1.27 1.27)) (justify right bottom))
-  )
   (label "D+" (at 294.64 195.58 0) (fields_autoplaced)
     (effects (font (size 1.27 1.27)) (justify left bottom))
@@
     (effects (font (size 1.27 1.27)) (justify right bottom))
   )
-  (label "P2" (at 312.42 58.42 180) (fields_autoplaced)
-    (effects (font (size 1.27 1.27)) (justify right bottom))
+  (label "MDI3_N" (at 253.365 99.06 0) (fields_autoplaced)
+    (effects (font (size 1.27 1.27)) (justify left bottom))
   )
   (label "SCL" (at 189.23 201.93 180) (fields_autoplaced)
     (effects (font (size 1.27 1.27)) (justify right bottom))
   )
-  (label "P10" (at 312.42 73.66 180) (fields_autoplaced)
-    (effects (font (size 1.27 1.27)) (justify right bottom))
+  (label "MDI2_N" (at 253.365 93.98 0) (fields_autoplaced)
+    (effects (font (size 1.27 1.27)) (justify left bottom))
   )
   (label "D+" (at 294.64 200.66 0) (fields_autoplaced)
     (effects (font (size 1.27 1.27)) (justify left bottom))
   )
+  (label "MDI3_N" (at 316.23 73.66 180) (fields_autoplaced)
+    (effects (font (size 1.27 1.27)) (justify right bottom))
+  )
   (label "A1" (at 106.68 225.425 180) (fields_autoplaced)
     (effects (font (size 1.27 1.27)) (justify right bottom))
   )
-  (label "P2" (at 256.54 83.82 0) (fields_autoplaced)
-    (effects (font (size 1.27 1.27)) (justify left bottom))
-  )
   (label "IN-" (at 148.59 212.09 0) (fields_autoplaced)
     (effects (font (size 1.27 1.27)) (justify left bottom))
   )
-  (label "P7" (at 256.54 91.44 0) (fields_autoplaced)
-    (effects (font (size 1.27 1.27)) (justify left bottom))
-  )
