File: USBPD_output.kicad_sch (KiCad schematic)
At the start: 43 parts, among them J2 Bus_RJ45_7499111121A, J3 USB-C_GCT_USB4105-GF-A, U10 TPD4E05U06QDQARQ1, U3 INA230AIRGTR, U6 TPS65987DDHRSHR

Commit message: Bump release date, unify naming
Other:
- note added: "Ethernet data output"
- note added: "USB Power Delivery output"
- note removed: "ETH out"
- note removed: "USBPD output"
Changed lines of the file:
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@@
 	(text "Drain1 and Drain2 are NC pins.\nWork as heat spreaders.\nKeep as big as possible."
 		(exclude_from_sim no)
-		(at 225.425 151.765 0)
+		(at 236.474 152.908 0)
 		(effects
 			(font
@@
 		)
 	)
-	(text "USBPD output"
+	(text "USB Power Delivery output"
 		(exclude_from_sim no)
 		(at 188.595 81.915 0)
@@
 		)
 	)
-	(text "ETH out"
+	(text "Ethernet data output"
 		(exclude_from_sim no)
 		(at 62.23 81.28 0)
